File: psu/eurorack1A_SMD/psu1A_smd.kicad_pcb (KiCad board)
At the start: 2 copper layers, 245.1 x 30.5 mm, 32 parts, among them J1 Conn_01x02_Male, J10 Conn_02x08_Odd_Even, J11 Conn_02x08_Odd_Even, J12 Conn_02x08_Odd_Even, J13 Conn_02x08_Odd_Even, J2 Conn_01x02_Male, J3 Conn_01x02_Male, J4 Conn_02x08_Odd_Even, J5 Conn_02x08_Odd_Even, J6 Conn_02x08_Odd_Even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

Commit message: SMD done
Parts:
- moved SW2 46.8 mm to (60.8, 57.4), turned to 270 degrees
- moved U2 42.3 mm to (109.0, 81.5), turned to 90 degrees
- moved R5 39.1 mm to (74.9, 55.3), turned to 180 degrees
- moved C6 37.9 mm to (134.7, 63.7), turned to 0 degrees
- moved C4 34.0 mm to (124.7, 59.7)
- moved C2 33.2 mm to (96.3, 58.7)
- moved H1 31.8 mm to (95.9, 71.1)
- moved R4 31.4 mm to (74.9, 62.1), turned to 180 degrees
- moved C5 29.8 mm to (120.5, 85.3)
- moved R1 28.3 mm to (74.9, 58.7)
- moved U1 27.9 mm to (64.6, 77.7)
- moved C1 27.9 mm to (96.3, 85.3), turned to 90 degrees
- moved J3 27.2 mm to (44.3, 54.9)
- moved D1 25.7 mm to (35.4, 85.3), turned to 180 degrees
- moved U4 25.5 mm to (126.8, 73.9), turned to 180 degrees
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Connections:
- SW2 pad 3: GND -> 0V
Routing:
- net -12V: track 144.7 -> 210.9 mm, vias 0 -> 2
- net +12V: track 155.5 -> 214.6 mm, vias 0 -> 2
- net Net-(J1-Pad1): track 0.00 -> 58.8 mm
- net VIN: track 0.00 -> 51.4 mm
- net +5V: track 242.3 -> 209.1 mm, vias 1 -> 2
- net Net-(R5-Pad2): track 0.00 -> 20.0 mm
- net Net-(R4-Pad2): track 0.00 -> 19.1 mm
- net Net-(R1-Pad2): track 0.00 -> 17.1 mm
- net -15V: track 18.3 -> 30.6 mm
- net +15V: track 17.8 -> 19.3 mm
- net 0V: track 0.11 -> 0.00 mm, vias 0 -> 195
- added copper zone on B.Cu, net 0V
Other:
- board size 245.1 x 30.5 mm -> 245.1 x 39.4 mm
