File: psu/eurorack1A_SMD/psu1A_smd.sch (KiCad schematic (older format))
At the start: 32 parts, among them J1 Conn_01x02_Male, J10 Conn_02x08_Odd_Even, J11 Conn_02x08_Odd_Even, J12 Conn_02x08_Odd_Even, J13 Conn_02x08_Odd_Even, J2 Conn_01x02_Male, J3 Conn_01x02_Male, J4 Conn_02x08_Odd_Even, J5 Conn_02x08_Odd_Even, J6 Conn_02x08_Odd_Even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

Commit message: SMD done
Connections:
- net 0V: now also SW2.3 (Pin_3)
- net GND: no longer SW2.3 (Pin_3)
Changed lines of the file:
@@
 Wire Wire Line
 	1600 1550 1850 1550
-Wire Wire Line
-	2250 1650 1950 1650
 $Comp
 L Device:R R1
@@
 Wire Wire Line
 	1600 4500 1500 4500
-Connection ~ 10450 1900
-Wire Wire Line
-	10450 1900 10700 1900
-Text GLabel 10700 1900 2    50   Input ~ 0
-0V
 Text GLabel 2300 4400 2    50   Input ~ 0
 0V
@@
 	1    0    0    -1
 $EndComp
-Connection ~ 1950 1650
 Text GLabel 4450 1550 0    50   Input ~ 0
 VIN
@@
 Text Notes 5100 2450 0    50   ~ 0
 DKMW30F-15\n(Different pinout, completly bollocks \npin numbering but compatible on the \nsecondary side, primary is done with vias.
+Text GLabel 2150 1650 0    50   Input ~ 0
+0V
+Wire Wire Line
+	2250 1650 2150 1650
 $EndSCHEMATC
